File: ESP32/cardspansion-esp.kicad_sch (KiCad schematic)
At the start: 5 parts, among them J1 M2-E 2230, U1 ESP32-WROOM-32UE, Y1 ASE-32.768KHZ

Commit message: Fix cardspansion-esp I2S wiring
I2S-SDIN and I2S-SDOUT nets were switched around
Connections:
- net I2S-SDIN: now also J1.12 (PCM_IN/I2S_SD_IN); no longer J1.14 (PCM_OUT/I2S_SD_OUT)
- net I2S-SDOUT: now also J1.14 (PCM_OUT/I2S_SD_OUT); no longer J1.12 (PCM_IN/I2S_SD_IN)
Changed lines of the file:
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@@
-		)
-	)
-	(label "I2S-SDIN"
-		(at 137.16 73.66 0)
-		(effects
-			(font
-				(size 1.27 1.27)
-			)
-			(justify left bottom)
 		)
 	)
@@
 		)
 	)
-	(label "I2S-SDOUT"
-		(at 137.16 71.12 0)
-		(effects
-			(font
-				(size 1.27 1.27)
-			)
-			(justify left bottom)
-		)
-	)
 	(label "UART-RX"
 		(at 54.61 50.8 0)
@@
 		)
 	)
+	(label "I2S-SDOUT"
+		(at 137.16 73.66 0)
+		(effects
+			(font
+				(size 1.27 1.27)
+			)
+			(justify left bottom)
+		)
+	)
 	(label "RTCIN"
 		(at 54.61 93.98 0)
@@
 		)
 	)
+	(label "I2S-SDIN"
+		(at 137.16 71.12 0)
+		(effects
+			(font
+				(size 1.27 1.27)
+			)
+			(justify left bottom)
+		)
+	)
