File: NRF53+NRF70/cardspansion-nrf.kicad_sch (KiCad schematic)
At the start: 4 parts, among them J1 M2-2230, U1 ME16WS03

Commit message: Fix cardspansion-nrf I2S wiring
I2S-SDIN and I2S-SDOUT nets were switched around
Connections:
- net I2S-SDIN: now also J1.12 (PCM_IN/I2S_SD_IN); no longer J1.14 (PCM_OUT/I2S_SD_OUT)
- net I2S-SDOUT: now also J1.14 (PCM_OUT/I2S_SD_OUT); no longer J1.12 (PCM_IN/I2S_SD_IN)
Changed lines of the file:
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@@
-		)
-	)
-	(label "I2S-SDIN"
-		(at 151.13 73.66 0)
-		(effects
-			(font
-				(size 1.27 1.27)
-			)
-			(justify left bottom)
 		)
 	)
@@
 		)
 	)
+	(label "I2S-SDIN"
+		(at 151.13 71.12 0)
+		(effects
+			(font
+				(size 1.27 1.27)
+			)
+			(justify left bottom)
+		)
+	)
 	(label "I2C-SCL"
 		(at 151.13 48.26 0)
@@
 			)
 			(justify right bottom)
+		)
+	)
+	(label "I2S-SDOUT"
+		(at 151.13 73.66 0)
+		(effects
+			(font
+				(size 1.27 1.27)
+			)
+			(justify left bottom)
 		)
 	)
@@
 		(effects
 			(font
-				(size 1.27 1.27)
-			)
-			(justify left bottom)
-		)
-	)
-	(label "I2S-SDOUT"
-		(at 151.13 71.12 0)
-		(effects
-			(font
